File: usbasp.kicad_pcb (KiCad board)
At the start: 2 copper layers, 54.9 x 19.6 mm, 25 parts, among them IC1 ATMEGA8A-P, P1 USB, P2 CONN_02X05, Y1 12MHz

Commit message: Add source code and some PCB changes
Parts:
- C1: footprint Capacitors_ThroughHole:C_Radial_D5_L6_P2.5 -> Capacitors_ThroughHole:CP_Radial_D5.0mm_P2.50mm
- D1, D2, D3: footprint Diodes_SMD:MELF_Standard -> Diodes_SMD:D_MiniMELF
- JP1, JP2, JP3, JP4: footprint Pin_Headers:Pin_Header_Straight_1x02 -> Pin_Headers:Pin_Header_Straight_1x02_Pitch2.54mm
- P2: footprint Pin_Headers:Pin_Header_Straight_2x05 -> Pin_Headers:Pin_Header_Straight_2x05_Pitch2.54mm
- moved D2 0.64 mm to (97.1, 90.6)
- moved D1 0.59 mm to (93.9, 83.4)
- moved D3 0.19 mm to (106.1, 79.2)
Routing:
- net Net-(D1-Pad1): track 7.38 -> 8.65 mm

Commit message: Update PCB
Parts:
- moved C4 5.01 mm to (120.8, 79.9), turned to 90 degrees
- moved P2 1.39 mm to (140.9, 82.0)
- moved R2 0.48 mm to (98.4, 80.6)
- moved R5 0.43 mm to (102.6, 88.1)
- moved R1 0.42 mm to (99.2, 84.4)
- moved R8 0.22 mm to (141.1, 78.9)
- moved R4 0.21 mm to (102.6, 85.7)
Routing:
- net GND: track 125.6 -> 100.7 mm
- net VCC: track 55.2 -> 63.7 mm
- net Net-(IC1-Pad2): track 22.7 -> 29.2 mm
- net Net-(IC1-Pad16): track 78.0 -> 80.4 mm
- net Net-(JP4-Pad2): track 15.2 -> 17.4 mm
- net Net-(IC1-Pad17): track 37.7 -> 39.5 mm
- net Net-(P2-Pad4): track 6.18 -> 7.90 mm
- net Net-(IC1-Pad19): track 28.9 -> 30.5 mm
- net Net-(D2-Pad1): track 10.3 -> 11.4 mm
- net Net-(IC1-Pad18): track 34.3 -> 35.3 mm
- net Net-(P1-Pad1): track 16.7 -> 15.8 mm
- net Net-(D5-Pad2): track 18.7 -> 19.6 mm
- net Net-(D1-Pad1): track 8.65 -> 7.95 mm
- net Net-(IC1-Pad14): track 2.85 -> 3.39 mm
Other:
- board size 54.9 x 19.6 mm -> 56.9 x 20.1 mm
