File: usbasp.sch (KiCad schematic (older format))
At the start: 25 parts, among them IC1 ATMEGA8A-P, P1 USB, P2 CONN_02X05, Y1 12MHz

Commit message: Add source code and some PCB changes
Parts:
- C1: footprint Capacitors_ThroughHole:C_Radial_D5_L6_P2.5 -> Capacitors_ThroughHole:CP_Radial_D5.0mm_P2.50mm
- D1, D2, D3: footprint Diodes_SMD:MELF_Standard -> Diodes_SMD:D_MiniMELF
- JP1, JP2, JP3, JP4: footprint Pin_Headers:Pin_Header_Straight_1x02 -> Pin_Headers:Pin_Header_Straight_1x02_Pitch2.54mm
- P2: footprint Pin_Headers:Pin_Header_Straight_2x05 -> Pin_Headers:Pin_Header_Straight_2x05_Pitch2.54mm
- Y1: value 12MHz -> 16.000
Changed lines of the file:
@@
 F 0 "D3" V 3300 3300 50  0000 L CNN
 F 1 "3.3v" V 3400 3300 50  0000 L CNN
-F 2 "Diodes_SMD:MELF_Standard" H 3450 3200 50  0001 C CNN
+F 2 "Diodes_SMD:D_MiniMELF" H 3450 3200 50  0001 C CNN
 F 3 "" H 3450 3200 50  0000 C CNN
 	1    3450 3200
@@
 F 0 "JP1" V 3300 3550 50  0000 L CNN
 F 1 "5/3.3v" V 3400 3550 50  0000 L CNN
-F 2 "Pin_Headers:Pin_Header_Straight_1x02" H 3450 3500 50  0001 C CNN
+F 2 "Pin_Headers:Pin_Header_Straight_1x02_Pitch2.54mm" H 3450 3500 50  0001 C CNN
 F 3 "" H 3450 3500 50  0000 C CNN
 	1    3450 3500
@@
 F 0 "C1" H 3850 3400 50  0000 L CNN
 F 1 "4.7" H 3850 3300 50  0000 L CNN
-F 2 "Capacitors_ThroughHole:C_Radial_D5_L6_P2.5" H 3800 3200 50  0001 C CNN
+F 2 "Capacitors_ThroughHole:CP_Radial_D5.0mm_P2.50mm" H 3800 3200 50  0001 C CNN
 F 3 "" H 3800 3200 50  0000 C CNN
 	1    3800 3200
@@
 F 0 "D1" V 2550 2750 50  0000 L CNN
 F 1 "3.3v" V 2650 2750 50  0000 L CNN
-F 2 "Diodes_SMD:MELF_Standard" H 2800 2700 50  0001 C CNN
+F 2 "Diodes_SMD:D_MiniMELF" H 2800 2700 50  0001 C CNN
 F 3 "" H 2800 2700 50  0000 C CNN
 	1    2800 2700
@@
 F 0 "D2" V 2800 2750 50  0000 L CNN
 F 1 "3.3v" V 2900 2750 50  0000 L CNN
-F 2 "Diodes_SMD:MELF_Standard" H 3050 2700 50  0001 C CNN
+F 2 "Diodes_SMD:D_MiniMELF" H 3050 2700 50  0001 C CNN
 F 3 "" H 3050 2700 50  0000 C CNN
 	1    3050 2700
@@
 F 0 "JP3" H 7000 3850 50  0000 C CNN
 F 1 "slow sck" H 7250 3850 50  0000 C CNN
-F 2 "Pin_Headers:Pin_Header_Straight_1x02" H 7000 3750 50  0001 C CNN
+F 2 "Pin_Headers:Pin_Header_Straight_1x02_Pitch2.54mm" H 7000 3750 50  0001 C CNN
 F 3 "" H 7000 3750 50  0000 C CNN
 	1    7000 3750
@@
 P 4400 3450
 F 0 "Y1" V 4100 3400 50  0000 L CNN
-F 1 "12MHz" V 4200 3400 50  0000 L CNN
+F 1 "16.000" V 4200 3400 50  0000 L CNN
 F 2 "Crystals:Crystal_HC50-U_Vertical" H 4400 3450 50  0001 C CNN
 F 3 "" H 4400 3450 50  0000 C CNN
@@
 F 0 "P2" H 8150 3350 50  0000 C CNN
 F 1 "CONN_02X05" H 8150 3250 50  0000 C CNN
-F 2 "Pin_Headers:Pin_Header_Straight_2x05" H 8150 1650 50  0001 C CNN
+F 2 "Pin_Headers:Pin_Header_Straight_2x05_Pitch2.54mm" H 8150 1650 50  0001 C CNN
 F 3 "" H 8150 1650 50  0000 C CNN
 	1    8150 2850
@@
 F 0 "JP2" V 6604 2624 50  0000 L CNN
 F 1 "Self programming" V 6695 2624 50  0000 L CNN
-F 2 "Pin_Headers:Pin_Header_Straight_1x02" H 6650 2550 50  0001 C CNN
+F 2 "Pin_Headers:Pin_Header_Straight_1x02_Pitch2.54mm" H 6650 2550 50  0001 C CNN
 F 3 "" H 6650 2550 50  0000 C CNN
 	1    6650 2550
@@
 F 0 "JP4" V 8604 2425 50  0000 L CNN
 F 1 "MC Power" V 8695 2425 50  0000 L CNN
-F 2 "Pin_Headers:Pin_Header_Straight_1x02" H 8650 2350 50  0001 C CNN
+F 2 "Pin_Headers:Pin_Header_Straight_1x02_Pitch2.54mm" H 8650 2350 50  0001 C CNN
 F 3 "" H 8650 2350 50  0000 C CNN
 	1    8650 2350

Commit message: Update PCB
Parts:
- C1: symbol CP_Small -> usbasp-rescue:CP_Small
- C2, C3, C4: symbol C_Small -> usbasp-rescue:C_Small
- D1, D2, D3: symbol D_Zener -> usbasp-rescue:D_Zener
- D4, D5: symbol LED -> usbasp-rescue:LED
- IC1: symbol ATMEGA8A-P -> atmel:ATMEGA8A-P
- JP1, JP2, JP3, JP4: symbol Jumper_NC_Small -> usbasp-rescue:Jumper_NC_Small
- P1: symbol CONN_01X05 -> usbasp-rescue:CONN_01X05
- P2: symbol CONN_02X05 -> usbasp-rescue:CONN_02X05
- R1, R2, R3, R4, R5, R6, R7, R8: symbol R -> usbasp-rescue:R
- Y1: symbol Crystal_Small -> usbasp-rescue:Crystal_Small
Changed lines of the file:
@@
-EESchema Schematic File Version 2
-LIBS:power
-LIBS:device
-LIBS:transistors
-LIBS:conn
-LIBS:linear
-LIBS:regul
-LIBS:74xx
-LIBS:cmos4000
-LIBS:adc-dac
-LIBS:memory
-LIBS:xilinx
-LIBS:microcontrollers
-LIBS:dsp
-LIBS:microchip
-LIBS:analog_switches
-LIBS:motorola
-LIBS:texas
-LIBS:intel
-LIBS:audio
-LIBS:interface
-LIBS:digital-audio
-LIBS:philips
-LIBS:display
-LIBS:cypress
-LIBS:siliconi
-LIBS:opto
-LIBS:atmel
-LIBS:contrib
-LIBS:valves
+EESchema Schematic File Version 4
 LIBS:usbasp-cache
 EELAYER 26 0
@@
 $EndDescr
 $Comp
-L ATMEGA8A-P IC1
+L atmel:ATMEGA8A-P IC1
 U 1 1 5852A98C
 P 5400 3750
@@
 $EndComp
 $Comp
-L CONN_01X05 P1
+L usbasp-rescue:CONN_01X05 P1
 U 1 1 5852AA4A
 P 2100 3200
@@
 $EndComp
 $Comp
-L R R2
+L usbasp-rescue:R R2
 U 1 1 5852AD51
 P 3250 3000
@@
 $EndComp
 $Comp
-L D_Zener D3
+L usbasp-rescue:D_Zener D3
 U 1 1 5852ADDE
 P 3450 3200
@@
 $EndComp
 $Comp
-L GND #PWR01
+L power:GND #PWR01
 U 1 1 5852AEF3
 P 2450 3650
@@
 $EndComp
 $Comp
-L VCC #PWR02
+L power:VCC #PWR02
 U 1 1 5852AFF3
 P 3450 2900
@@
 $EndComp
 $Comp
-L Jumper_NC_Small JP1
+L usbasp-rescue:Jumper_NC_Small JP1
 U 1 1 5852B089
 P 3450 3500
@@
 $EndComp
 $Comp
-L GND #PWR03
+L power:GND #PWR03
 U 1 1 5852B0E8
 P 3450 3650
@@
 $EndComp
 $Comp
-L CP_Small C1
+L usbasp-rescue:CP_Small C1
 U 1 1 5852B1AF
 P 3800 3200
@@
 $EndComp
 $Comp
-L GND #PWR04
+L power:GND #PWR04
 U 1 1 5852B211
 P 3800 3650
@@
 $EndComp
 $Comp
-L R R4
+L usbasp-rescue:R R4
 U 1 1 5852B2FE
 P 6200 1950
@@
 $EndComp
 $Comp
-L R R5
+L usbasp-rescue:R R5
 U 1 1 5852B40A
 P 6200 2150
@@
 $EndComp
 $Comp
-L VCC #PWR05
+L power:VCC #PWR05
 U 1 1 5852B710
 P 5400 1850
@@
 $EndComp
 $Comp
-L C_Small C4
+L usbasp-rescue:C_Small C4
 U 1 1 5852B779
 P 3000 5150
@@
 $EndComp
 $Comp
-L GND #PWR06
+L power:GND #PWR06
 U 1 1 5852B7B3
 P 3000 5300
@@
 $EndComp
 $Comp
-L R R1
+L usbasp-rescue:R R1
 U 1 1 5852B999
 P 2600 2700
@@
 $EndComp
 $Comp
-L D_Zener D1
+L usbasp-rescue:D_Zener D1
 U 1 1 5852BC1C
 P 2800 2700
@@
 $EndComp
 $Comp
-L D_Zener D2
+L usbasp-rescue:D_Zener D2
 U 1 1 5852BD51
 P 3050 2700
@@
 $EndComp
 $Comp
-L GND #PWR07
+L power:GND #PWR07
 U 1 1 5852BE18
 P 2800 3650
@@
 $EndComp
 $Comp
-L GND #PWR08
+L power:GND #PWR08
 U 1 1 5852BE44
 P 3050 3650
@@
 $EndComp
 $Comp
-L LED D4
+L usbasp-rescue:LED D4
 U 1 1 5852C568
 P 6950 3350
@@
 $EndComp
 $Comp
-L LED D5
+L usbasp-rescue:LED D5
 U 1 1 5852C7DE
 P 6950 3550
@@
 $EndComp
 $Comp
-L R R6
+L usbasp-rescue:R R6
 U 1 1 5852C9BA
 P 7450 3350
@@
 $EndComp
 $Comp
-L R R7
+L usbasp-rescue:R R7
 U 1 1 5852CA16
 P 7450 3550
@@
 $EndComp
 $Comp
-L VCC #PWR09
+L power:VCC #PWR09
 U 1 1 5852CBB8
 P 7650 2100
@@
 $EndComp
 $Comp
-L Jumper_NC_Small JP3
+L usbasp-rescue:Jumper_NC_Small JP3
 U 1 1 5852D760
 P 7000 3750
@@
 $EndComp
 $Comp
-L GND #PWR010
+L power:GND #PWR010
 U 1 1 5852D903
 P 7650 3800
@@
 $EndComp
 $Comp
-L Crystal_Small Y1
+L usbasp-rescue:Crystal_Small Y1
 U 1 1 5852DDF8
 P 4400 3450
@@
 $EndComp
 $Comp
-L C_Small C2
+L usbasp-rescue:C_Small C2
 U 1 1 5852DF89
 P 4150 3350
@@
 $EndComp
 $Comp
-L C_Small C3
+L usbasp-rescue:C_Small C3
 U 1 1 5852DFF9
 P 4150 3550
@@
 $EndComp
 $Comp
-L GND #PWR011
+L power:GND #PWR011
 U 1 1 5852E207
 P 4000 3650
@@
 $EndComp
 $Comp
-L R R3
+L usbasp-rescue:R R3
 U 1 1 5852E86B
 P 4250 2650
@@
 $EndComp
 $Comp
-L VCC #PWR012
+L power:VCC #PWR012
 U 1 1 5852E900
 P 4000 2550
@@
 $EndComp
 $Comp
-L CONN_02X05 P2
+L usbasp-rescue:CONN_02X05 P2
 U 1 1 5853B12C
 P 8150 2850
@@
 $EndComp
 $Comp
-L GND #PWR013
+L power:GND #PWR013
 U 1 1 5853BD07
 P 8450 3800
@@
 $EndComp
 $Comp
-L R R8
+L usbasp-rescue:R R8
 U 1 1 5853BE97
 P 7450 4150
@@
 $EndComp
 $Comp
-L Jumper_NC_Small JP2
+L usbasp-rescue:Jumper_NC_Small JP2
 U 1 1 5853C3DC
 P 6650 2550
@@
 $EndComp
 $Comp
-L Jumper_NC_Small JP4
+L usbasp-rescue:Jumper_NC_Small JP4
 U 1 1 5853C555
 P 8650 2350
@@
 $EndComp
 $Comp
-L VCC #PWR014
+L power:VCC #PWR014
 U 1 1 5853C99B
 P 8650 2100
@@
 $EndComp
 Wire Wire Line
-	2300 3000 3100 3000
-Wire Wire Line
-	3450 2900 3450 3050
-Wire Wire Line
-	3400 3000 3800 3000
-Wire Wire Line
-	2450 3300 2450 3650
+	2300 3000 2600 3000
+Wire Wire Line
+	3450 2900 3450 3000
+Wire Wire Line
+	3400 3000 3450 3000
+Wire Wire Line
+	2450 3300 2450 3400
 Connection ~ 3450 3000
 Wire Wire Line
@@
 	6550 2650 6400 2650
 Wire Wire Line
-	2350 1950 6050 1950
-Wire Wire Line
-	2350 1950 2350 3100
+	2350 1950 2800 1950
+Wire Wire Line
+	2350 1950 2350 2500
 Wire Wire Line
 	2350 3100 2300 3100
 Wire Wire Line
-	2450 2150 6050 2150
+	2450 2150 3050 2150
 Wire Wire Line
 	2450 2150 2450 3200
@@
 	6350 2150 6450 2150
 Wire Wire Line
-	6450 2150 6450 4250
+	6450 2150 6450 2750
 Wire Wire Line
 	6450 4250 6400 4250
@@
 	7600 3350 7650 3350
 Wire Wire Line
-	7650 2100 7650 3550
+	7650 2100 7650 3350
 Wire Wire Line
 	7650 3550 7600 3550
@@
 	6550 3550 6400 3550
 Wire Wire Line
-	4250 3550 4500 3550
+	4250 3550 4400 3550
 Connection ~ 4400 3550
 Wire Wire Line
-	4250 3350 4500 3350
+	4250 3350 4400 3350
 Connection ~ 4400 3350
 Wire Wire Line
 	4050 3350 4000 3350
 Wire Wire Line
-	4000 3050 4000 3650
+	4000 3050 4000 3350
 Wire Wire Line
 	4000 3550 4050 3550
 Connection ~ 4000 3550
 Wire Wire Line
-	4000 2550 4000 2850
+	4000 2550 4000 2650
 Wire Wire Line
 	4000 2650 4100 2650
 Wire Wire Line
-	4400 2650 4500 2650
+	4400 2650 4450 2650
 Wire Wire Line
 	4500 3050 4000 3050
@@
 	7850 2950 7900 2950
 Wire Wire Line
-	6400 2850 7900 2850
+	6400 2850 6650 2850
 Wire Wire Line
 	6400 2950 7750 2950
@@
 	7750 2650 7900 2650
 Wire Wire Line
-	8450 2500 8450 3800
+	8450 2500 8450 2950
 Wire Wire Line
 	8450 2950 8400 2950
@@
 	8650 2100 8650 2250
 $Comp
-L GND #PWR015
+L power:GND #PWR015
 U 1 1 58540035
 P 5400 5300
@@
 Connection ~ 8450 2950
 $Comp
-L VCC #PWR016
+L power:VCC #PWR016
 U 1 1 58543551
 P 3000 5000
@@
 Wire Wire Line
 	3000 5250 3000 5300
+Wire Wire Line
+	3450 3000 3450 3050
+Wire Wire Line
+	3450 3000 3800 3000
+Wire Wire Line
+	6450 2750 6450 4250
+Wire Wire Line
+	2450 3400 2450 3650
+Wire Wire Line
+	3050 2150 6050 2150
+Wire Wire Line
+	2800 1950 6050 1950
+Wire Wire Line
+	7650 3350 7650 3550
+Wire Wire Line
+	4400 3550 4500 3550
+Wire Wire Line
+	4400 3350 4500 3350
+Wire Wire Line
+	4000 3550 4000 3650
+Wire Wire Line
+	4000 2650 4000 2850
+Wire Wire Line
+	4000 3350 4000 3550
+Wire Wire Line
+	8450 3050 8450 3800
+Wire Wire Line
+	4450 2650 4500 2650
+Wire Wire Line
+	6650 2850 7900 2850
+Wire Wire Line
+	2600 3000 3100 3000
+Wire Wire Line
+	2350 2500 2350 3100
+Wire Wire Line
+	8450 2950 8450 3050
 $EndSCHEMATC
